File: PCB/PCB.kicad_pcb (KiCad board)
At the start: 2 copper layers, 82.5 x 100 mm, 37 parts, among them SW1 SW_Push, SW10 SW_Push, SW11 SW_Push, SW12 SW_Push, SW13 RotaryEncoder_Switch, SW2 SW_Push, SW3 SW_Push, SW4 SW_Push, SW5 SW_Push, SW6 SW_Push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

Commit message: Add files via upload
Parts:
- D13, D14, D15, D16, D17: value WS2812B -> SK6812; footprint LED_SMD:LED_WS2812B_PLCC4_5.0x5.0mm_P3.2mm -> LED_SMD:LED_SK6812_PLCC4_5.0x5.0mm_P3.2mm
- moved D15 82.8 mm to (130.3, 86.0)
- moved D13 82.7 mm to (191.1, 29.2)
- moved D14 61.9 mm to (190.1, 84.7)
- moved D17 61.7 mm to (130.1, 104.2)
- moved D16 16.3 mm to (190.1, 103.7)
- moved D18 4.00 mm to (142.1, 33.5)
Connections:
- D13 pad 1: GND -> VCC
- D13 pad 2: Net-(D13-DOUT) -> WS2812B
- D13 pad 3: VCC -> GND
- D13 pad 4: WS2812B -> unconnected-(D13-DOUT-Pad4)
- D14 pad 1: GND -> VCC
- D14 pad 2: unconnected-(D14-DOUT-Pad2) -> Net-(D14-DIN)
- D14 pad 3: VCC -> GND
- D14 pad 4: Net-(D13-DOUT) -> unconnected-(D14-DOUT-Pad4)
- D15 pad 1: GND -> VCC
- D15 pad 2: unconnected-(D15-DOUT-Pad2) -> Net-(D15-DIN)
- D15 pad 3: VCC -> GND
- D15 pad 4: WS2812B -> unconnected-(D15-DOUT-Pad4)
- D16 pad 1: GND -> VCC
- D16 pad 2: Net-(D16-DOUT) -> WS2812B
- D16 pad 3: VCC -> GND
- D16 pad 4: WS2812B -> Net-(D14-DIN)
- D17 pad 1: GND -> VCC
- D17 pad 2: unconnected-(D17-DOUT-Pad2) -> WS2812B
- D17 pad 3: VCC -> GND
- D17 pad 4: Net-(D16-DOUT) -> Net-(D15-DIN)
Routing:
- net Net-(D16-DOUT): track 20.0 -> 0.00 mm
- net Net-(D14-DIN): track 0.00 -> 17.8 mm, vias 0 -> 2
- net Net-(D13-DOUT): track 17.6 -> 0.00 mm, vias 2 -> 0
- net Net-(D15-DIN): track 0.00 -> 16.9 mm
- net VCC: track 170.2 -> 180.6 mm, vias 4 -> 2
- net GND: track 186.6 -> 177.9 mm, vias 2 -> 6
- net WS2812B: track 145.9 -> 149.9 mm

Commit message: Add files via upload
Parts:
- D13, D14, D15, D16, D17: footprint LED_SMD:LED_SK6812_PLCC4_5.0x5.0mm_P3.2mm -> LED_SMD:LED_SK6812MINI_PLCC4_3.5x3.5mm_P1.75mm
Routing:
- net GND: track 177.9 -> 181.9 mm
- net Net-(D14-DIN): track 17.8 -> 19.8 mm
- net WS2812B: track 149.9 -> 151.5 mm
- net VCC: track 180.6 -> 182.2 mm
- net Net-(D15-DIN): track 16.9 -> 18.4 mm
- removed copper zone on B.Cu, net (none)
- removed copper zone on F.Cu, net (none)

Commit message: Add files via upload
Connections:
- D13 pad 1: VCC -> GND
- D13 pad 2: WS2812B -> unconnected-(D13-DOUT-Pad2)
- D13 pad 3: GND -> VCC
- D13 pad 4: unconnected-(D13-DOUT-Pad4) -> SK6812
- D14 pad 1: VCC -> GND
- D14 pad 2: Net-(D14-DIN) -> unconnected-(D14-DOUT-Pad2)
- D14 pad 3: GND -> VCC
- D14 pad 4: unconnected-(D14-DOUT-Pad4) -> Net-(D14-DIN)
- D15 pad 1: VCC -> GND
- D15 pad 2: Net-(D15-DIN) -> unconnected-(D15-DOUT-Pad2)
- D15 pad 3: GND -> VCC
- D15 pad 4: unconnected-(D15-DOUT-Pad4) -> Net-(D15-DIN)
- D16 pad 1: VCC -> GND
- D16 pad 2: WS2812B -> Net-(D14-DIN)
- D16 pad 3: GND -> VCC
- D16 pad 4: Net-(D14-DIN) -> SK6812
- D17 pad 1: VCC -> GND
- D17 pad 2: WS2812B -> Net-(D15-DIN)
- D17 pad 3: GND -> VCC
- D17 pad 4: Net-(D15-DIN) -> SK6812
- U1 pad 11: WS2812B -> SK6812
Routing:
- net SK6812: track 0.00 -> 211.3 mm, vias 0 -> 4
- net WS2812B: track 151.5 -> 0.00 mm, vias 2 -> 0
- net GND: track 181.9 -> 188.0 mm
- net Net-(D14-DIN): track 19.8 -> 23.9 mm
- net Net-(D15-DIN): track 18.4 -> 21.5 mm
- net VCC: track 182.2 -> 183.3 mm, vias 2 -> 1
- added copper zone on B.Cu, net (none)
- added copper zone on F.Cu, net (none)

Commit message: Add files via upload
Parts:
- D16: footprint LED_SMD:LED_SK6812MINI_PLCC4_3.5x3.5mm_P1.75mm -> footprints:SK6812MINI-E_fixed
Routing:
- net VCC: track 183.3 -> 206.9 mm
- net EC11B: track 86.8 -> 91.6 mm
- net GND: track 188.0 -> 183.5 mm
- net SK6812: track 211.3 -> 207.3 mm
- net Net-(D14-DIN): track 23.9 -> 20.3 mm, vias 2 -> 0
- net Net-(D15-DIN): track 21.5 -> 19.1 mm
- removed copper zone on B.Cu, net (none)
- removed copper zone on F.Cu, net (none)

Commit message: Add files via upload
Routing:
- net GND: track 183.5 -> 168.4 mm, vias 6 -> 2
- net VCC: track 206.9 -> 220.3 mm, vias 1 -> 2
- net SK6812: track 207.3 -> 202.9 mm, vias 4 -> 3
